File: pcb/kicad/RevF/fpga.sch (KiCad schematic (older format))
At the start: 25 parts, among them P113 CONN_1, U201 XC3S400-PQ208

Commit message: S-DD1 + base (trick)
"sd2snes_trick" is the same implementation than "sd2snes_sdd1" but it is
intended to be used as base firmware. It implements S-DD1 core but it is
always disabled. It loads ROMs and runs games perfectly, except for
StarOcean.
"sd2snes_sdd1" corrects BHE and BLE assertion so all accesses from S-DD1
to PSRAM are 16bit wide.
"main.v" simulation is successfull and we get decompressed graphics as
output.
Parts:
- C201, C202, C203, C204, C205, C206, C207, C208, C209, C210, C211, C212, C213, C214, C215, C221, C222, C223, C224, C231, C232, C233, C234: symbol C -> Device:C
Changed lines of the file:
@@
-EESchema Schematic File Version 2
-LIBS:power
-LIBS:device
-LIBS:transistors
-LIBS:conn
-LIBS:linear
-LIBS:regul
-LIBS:74xx
-LIBS:cmos4000
-LIBS:adc-dac
-LIBS:memory
-LIBS:xilinx
-LIBS:special
-LIBS:microcontrollers
-LIBS:dsp
-LIBS:microchip
-LIBS:analog_switches
-LIBS:motorola
-LIBS:texas
-LIBS:intel
-LIBS:audio
-LIBS:interface
-LIBS:digital-audio
-LIBS:philips
-LIBS:display
-LIBS:cypress
-LIBS:siliconi
-LIBS:opto
-LIBS:atmel
-LIBS:contrib
-LIBS:valves
-LIBS:snescart
-LIBS:misc-74
-LIBS:vreg
-LIBS:lpc1754
-LIBS:sd_card
-LIBS:cy62148ev30
-LIBS:mt45w8mw16
-LIBS:cs4344
-LIBS:double_sch_kcom
-LIBS:usb_minib
-LIBS:mic23250
-LIBS:sd2snes-cache
-EELAYER 27 0
+EESchema Schematic File Version 4
+EELAYER 26 0
 EELAYER END
 $Descr A3 16535 11693
@@
 Connection ~ 3400 10350
 $Comp
-L C C234
+L Device:C C234
 U 1 1 4D2F566A
 P 3650 10650
@@
 $EndComp
 $Comp
-L C C233
+L Device:C C233
 U 1 1 4D2F497B
 P 3400 10650
@@
 $EndComp
 $Comp
-L C C232
+L Device:C C232
 U 1 1 4D2F4979
 P 3150 10650
@@
 $EndComp
 $Comp
-L C C215
+L Device:C C215
 U 1 1 4D2F4480
 P 5350 10650
@@
 $EndComp
 $Comp
-L C C231
+L Device:C C231
 U 1 1 4D2F4344
 P 2900 10650
@@
 $EndComp
 $Comp
-L C C209
+L Device:C C209
 U 1 1 4D2F4312
 P 2650 10650
@@
 $EndComp
 $Comp
-L C C214
+L Device:C C214
 U 1 1 4D252B5C
 P 5100 10650
@@
 DAC
 $Comp
-L C C224
+L Device:C C224
 U 1 1 4BF5A441
 P 6400 10650
@@
 $EndComp
 $Comp
-L C C223
+L Device:C C223
 U 1 1 4BF5A43F
 P 6150 10650
@@
 SNES_SYS_CLK
 $Comp
-L GND #PWR0113
+L power:GND #PWR0113
 U 1 1 4BADE94E
 P 5800 2000
@@
 $EndComp
 $Comp
-L GND #PWR0114
+L power:GND #PWR0114
 U 1 1 4BADE8CE
 P 8450 10900
@@
 $EndComp
 $Comp
-L GND #PWR0117
+L power:GND #PWR0117
 U 1 1 4BADD08B
 P 5650 11100
@@
 $EndComp
 $Comp
-L GND #PWR0118
+L power:GND #PWR0118
 U 1 1 4BADD089
 P 4100 11100
@@
 $EndComp
 $Comp
-L GND #PWR0119
+L power:GND #PWR0119
 U 1 1 4BADD072
 P 650 11100
@@
 $EndComp
 $Comp
-L +3.3V #PWR0120
+L power:+3.3V #PWR0120
 U 1 1 4BADD05C
 P 650 10200
@@
 $EndComp
 $Comp
-L C C222
+L Device:C C222
 U 1 1 4BADCE85
 P 5900 10650
@@
 $EndComp
 $Comp
-L C C221
+L Device:C C221
 U 1 1 4BADCE7D
 P 5650 10650
@@
 $EndComp
 $Comp
-L C C213
+L Device:C C213
 U 1 1 4BADCE7B
 P 4850 10650
@@
 $EndComp
 $Comp
-L C C212
+L Device:C C212
 U 1 1 4BADCE7A
 P 4600 10650
@@
 $EndComp
 $Comp
-L C C211
+L Device:C C211
 U 1 1 4BADCE78
 P 4350 10650
@@
 $EndComp
 $Comp
-L C C210
+L Device:C C210
 U 1 1 4BADCE74
 P 4100 10650
@@
 $EndComp
 $Comp
-L C C208
+L Device:C C208
 U 1 1 4BADCE6D
 P 2400 10650
@@
 $EndComp
 $Comp
-L C C207
+L Device:C C207
 U 1 1 4BADCE6B
 P 2150 10650
@@
 $EndComp
 $Comp
-L C C206
+L Device:C C206
 U 1 1 4BADCE6A
 P 1900 10650
@@
 $EndComp
 $Comp
-L C C205
+L Device:C C205
 U 1 1 4BADCE67
 P 1650 10650
@@
 $EndComp
 $Comp
-L C C204
+L Device:C C204
 U 1 1 4BADCE65
 P 1400 10650
@@
 $EndComp
 $Comp
-L C C203
+L Device:C C203
 U 1 1 4BADCE64
 P 1150 10650
@@
 $EndComp
 $Comp
-L C C202
+L Device:C C202
 U 1 1 4BADCE62
 P 900 10650
@@
 $EndComp
 $Comp
-L C C201
+L Device:C C201
 U 1 1 4BADCE47
 P 650 10650
@@
 JTAG
 $Comp
-L +3.3V #PWR0121
+L power:+3.3V #PWR0121
 U 1 1 4BAD12D2
 P 7650 800
