File: pcb/kicad/RevF/mcu.sch (KiCad schematic (older format))
At the start: 35 parts, among them J411 Hirose DM1AA, J421 USB Mini-B SMT, P401 CONN_7X2, P402 CONN_2, P403 CONN_2, P404 CONN_3X2, U401 LPC1754, X401 12MHz, X402 32.768kHz

Commit message: S-DD1 + base (trick)
"sd2snes_trick" is the same implementation than "sd2snes_sdd1" but it is
intended to be used as base firmware. It implements S-DD1 core but it is
always disabled. It loads ROMs and runs games perfectly, except for
StarOcean.
"sd2snes_sdd1" corrects BHE and BLE assertion so all accesses from S-DD1
to PSRAM are 16bit wide.
"main.v" simulation is successfull and we get decompressed graphics as
output.
Parts:
- C401, C402, C403, C404, C405, C406, C407, C408, C409, C411, C412: symbol C -> Device:C
- D401, D402, D403: symbol LED -> Device:LED
- J411: symbol SD_CARD -> sd_card:SD_CARD
- J421: symbol USB_MINIB -> usb_minib:USB_MINIB
- JP401, JP402: symbol JUMPER -> Device:Jumper
- R401, R402, R403, R404, R405, R406, R407, R421, R422, R423: symbol R -> Device:R
- U401: symbol LPC1754 -> lpc1754:LPC1754
- X401, X402: symbol CRYSTAL -> Device:Crystal
Changed lines of the file:
@@
-EESchema Schematic File Version 2
-LIBS:power
-LIBS:device
-LIBS:transistors
-LIBS:conn
-LIBS:linear
-LIBS:regul
-LIBS:74xx
-LIBS:cmos4000
-LIBS:adc-dac
-LIBS:memory
-LIBS:xilinx
-LIBS:special
-LIBS:microcontrollers
-LIBS:dsp
-LIBS:microchip
-LIBS:analog_switches
-LIBS:motorola
-LIBS:texas
-LIBS:intel
-LIBS:audio
-LIBS:interface
-LIBS:digital-audio
-LIBS:philips
-LIBS:display
-LIBS:cypress
-LIBS:siliconi
-LIBS:opto
-LIBS:atmel
-LIBS:contrib
-LIBS:valves
-LIBS:snescart
-LIBS:misc-74
-LIBS:vreg
-LIBS:lpc1754
-LIBS:sd_card
-LIBS:cy62148ev30
-LIBS:mt45w8mw16
-LIBS:cs4344
-LIBS:double_sch_kcom
-LIBS:usb_minib
-LIBS:mic23250
-LIBS:sd2snes-cache
-EELAYER 27 0
+EESchema Schematic File Version 4
+EELAYER 26 0
 EELAYER END
 $Descr A4 11693 8268
@@
 	6700 5000 7950 5000
 $Comp
-L GND #PWR045
+L power:GND #PWR045
 U 1 1 4E2C17DC
 P 4200 7400
@@
 /USEBATT
 $Comp
-L JUMPER JP402
+L Device:Jumper JP402
 U 1 1 4E2C1796
 P 4700 7200
@@
 open in case of in-circuit PIC programming
 $Comp
-L JUMPER JP401
+L Device:Jumper JP401
 U 1 1 4C86265B
 P 7300 5950
@@
 $EndComp
 $Comp
-L R R407
+L Device:R R407
 U 1 1 4C814430
 P 1400 3700
@@
 $EndComp
 $Comp
-L +3.3V #PWR046
+L power:+3.3V #PWR046
 U 1 1 4C814422
 P 1400 3400
@@
 NoConn ~ 3200 2500
 $Comp
-L R R422
+L Device:R R422
 U 1 1 4C5608C9
 P 7450 4200
@@
 $EndComp
 $Comp
-L R R421
+L Device:R R421
 U 1 1 4C5608C6
 P 7450 4100
@@
 $EndComp
 $Comp
-L GND #PWR047
+L power:GND #PWR047
 U 1 1 4C4A0B6E
 P 7950 6700
@@
 DIN+MCU_/OVR
 $Comp
-L C C412
+L Device:C C412
 U 1 1 4C1286D5
 P 10950 3100
@@
 $EndComp
 $Comp
-L LED D403
+L Device:LED D403
 U 1 1 4C0DA78D
 P 800 2500
@@
 $EndComp
 $Comp
-L R R403
+L Device:R R403
 U 1 1 4C0DA785
 P 2000 3200
@@
 2mA low current LEDs
 $Comp
-L C C405
+L Device:C C405
 U 1 1 4C063C47
 P 1400 5600
@@
 $EndComp
 $Comp
-L R R404
+L Device:R R404
 U 1 1 4C063C2F
 P 1400 4900
@@
 $EndComp
 $Comp
-L +3.3V #PWR048
+L power:+3.3V #PWR048
 U 1 1 4C063C16
 P 1400 4600
@@
 $EndComp
 $Comp
-L R R423
+L Device:R R423
 U 1 1 4C01596A
 P 9300 5000
@@
 /RESET
 $Comp
-L +5V #PWR049
+L power:+5V #PWR049
 U 1 1 4BFBFF63
 P 10500 5750
@@
 $EndComp
 $Comp
-L +3.3V #PWR050
+L power:+3.3V #PWR050
 U 1 1 4BFBFF50
 P 9200 5750
@@
 $EndComp
 $Comp
-L GND #PWR051
+L power:GND #PWR051
 U 1 1 4BFBFF44
 P 8850 5850
@@
 TX3
 $Comp
-L R R405
+L Device:R R405
 U 1 1 4BF850D1
 P 7250 3300
@@
 $EndComp
 $Comp
-L R R406
+L Device:R R406
 U 1 1 4BF850A9
 P 7450 5100
@@
 $EndComp
 $Comp
-L +3.3V #PWR052
+L power:+3.3V #PWR052
 U 1 1 4BF84ABB
 P 1100 1900
@@
 $EndComp
 $Comp
-L R R402
+L Device:R R402
 U 1 1 4BF847B1
 P 2000 3100
@@
 $EndComp
 $Comp
-L R R401
+L Device:R R401
 U 1 1 4BF847A7
 P 2000 3000
@@
 $EndComp
 $Comp
-L LED D401
+L Device:LED D401
 U 1 1 4BF8328D
 P 1400 2500
@@
 $EndComp
 $Comp
-L LED D402
+L Device:LED D402
 U 1 1 4BF8324A
 P 1100 2500
@@
 $EndComp
 $Comp
-L GND #PWR053
+L power:GND #PWR053
 U 1 1 4BF6C1FC
 P 5850 7600
@@
 $EndComp
 $Comp
-L +3.3V #PWR054
+L power:+3.3V #PWR054
 U 1 1 4BF6C1F7
 P 5850 6800
@@
 $EndComp
 $Comp
-L C C404
+L Device:C C404
 U 1 1 4BF6BFE6
 P 6600 7200
@@
 $EndComp
 $Comp
-L C C403
+L Device:C C403
 U 1 1 4BF6BFE5
 P 6350 7200
@@
 $EndComp
 $Comp
-L C C402
+L Device:C C402
 U 1 1 4BF6BFE2
 P 6100 7200
@@
 $EndComp
 $Comp
-L C C401
+L Device:C C401
 U 1 1 4BF6BFE1
 P 5850 7200
@@
 $EndComp
 $Comp
-L C C411
+L Device:C C411
 U 1 1 4BF6BFBB
 P 10700 3100
@@
 CIC_DATA1
 $Comp
-L GND #PWR055
+L power:GND #PWR055
 U 1 1 4BF0021F
 P 9600 5200
@@
 $EndComp
 $Comp
-L USB_MINIB J421
+L usb_minib:USB_MINIB J421
 U 1 1 4BF00175
 P 10100 4700
@@
 $EndComp
 $Comp
-L GND #PWR056
+L power:GND #PWR056
 U 1 1 4BEFBCAA
 P 1200 6850
@@
 DONE
 $Comp
-L SD_CARD J411
+L sd_card:SD_CARD J411
 U 1 1 4BAA6A9C
 P 9650 3250
@@
 CIC_MCLR
 $Comp
-L GND #PWR057
+L power:GND #PWR057
 U 1 1 4BEECBF1
 P 3100 6850
@@
 $EndComp
 $Comp
-L GND #PWR058
+L power:GND #PWR058
 U 1 1 4BEECBEF
 P 2500 6850
@@
 $EndComp
 $Comp
-L GND #PWR059
+L power:GND #PWR059
 U 1 1 4BEECBEE
 P 2200 6850
@@
 $EndComp
 $Comp
-L GND #PWR060
+L power:GND #PWR060
 U 1 1 4BEECBE5
 P 1600 6850
@@
 $EndComp
 $Comp
-L C C409
+L Device:C C409
 U 1 1 4BEECBD1
 P 3100 6600
@@
 $EndComp
 $Comp
-L C C408
+L Device:C C408
 U 1 1 4BEECBCD
 P 2500 6600
@@
 $EndComp
 $Comp
-L C C407
+L Device:C C407
 U 1 1 4BEECBCA
 P 2200 6600
@@
 $EndComp
 $Comp
-L C C406
+L Device:C C406
 U 1 1 4BEECBC1
 P 1600 6600
@@
 SD_CLK
 $Comp
-L CRYSTAL X402
+L Device:Crystal X402
 U 1 1 4BC243CB
 P 2800 6200
@@
 $EndComp
 $Comp
-L CRYSTAL X401
+L Device:Crystal X401
 U 1 1 4BC243C8
 P 1900 6200
@@
 $EndComp
 $Comp
-L GND #PWR061
+L power:GND #PWR061
 U 1 1 4BB8BBE8
 P 10700 3900
@@
 $EndComp
 $Comp
-L +3.3V #PWR062
+L power:+3.3V #PWR062
 U 1 1 4BB8BBD6
 P 10700 2650
@@
 $EndComp
 $Comp
-L +3.3V #PWR063
+L power:+3.3V #PWR063
 U 1 1 4BB8BB64
 P 4650 1450
@@
 $EndComp
 $Comp
-L GND #PWR064
+L power:GND #PWR064
 U 1 1 4BB8BB56
 P 4450 6850
@@
 $EndComp
 $Comp
-L +BATT #PWR065
+L power:+BATT #PWR065
 U 1 1 4BB8AE61
 P 4350 1450
@@
 $EndComp
 $Comp
-L +3.3V #PWR066
+L power:+3.3V #PWR066
 U 1 1 4BB8AE12
 P 5250 1450
@@
 $EndComp
 $Comp
-L GND #PWR067
+L power:GND #PWR067
 U 1 1 4BAF2DEB
 P 4650 6850
@@
 $EndComp
 $Comp
-L GND #PWR068
+L power:GND #PWR068
 U 1 1 4BAF2DE3
 P 5100 6850
@@
 $EndComp
 $Comp
-L LPC1754 U401
+L lpc1754:LPC1754 U401
 U 1 1 4B6F321A
 P 5000 4100
