File: pcb/kicad/RevF/memory.sch (KiCad schematic (older format))
At the start: 10 parts, among them Q511 2N2222A, U501 MT45W8MW16, U511 CY62148EV30-ZSXI

Commit message: S-DD1 + base (trick)
"sd2snes_trick" is the same implementation than "sd2snes_sdd1" but it is
intended to be used as base firmware. It implements S-DD1 core but it is
always disabled. It loads ROMs and runs games perfectly, except for
StarOcean.
"sd2snes_sdd1" corrects BHE and BLE assertion so all accesses from S-DD1
to PSRAM are 16bit wide.
"main.v" simulation is successfull and we get decompressed graphics as
output.
Parts:
- C501, C502, C511: symbol C -> Device:C
- D511: symbol DOUBLE_SCH_KCOM2 -> double_sch_kcom:DOUBLE_SCH_KCOM2
- R511, R512, R513: symbol R -> Device:R
- U501: symbol MT45W8MW16 -> mt45w8mw16:MT45W8MW16
- U511: symbol CY62148EV30-ZSXI -> cy62148ev30:CY62148EV30-ZSXI
Connections:
- wire segments 105 -> 112
Changed lines of the file:
@@
-EESchema Schematic File Version 2
-LIBS:power
-LIBS:device
-LIBS:transistors
-LIBS:conn
-LIBS:linear
-LIBS:regul
-LIBS:74xx
-LIBS:cmos4000
-LIBS:adc-dac
-LIBS:memory
-LIBS:xilinx
-LIBS:special
-LIBS:microcontrollers
-LIBS:dsp
-LIBS:microchip
-LIBS:analog_switches
-LIBS:motorola
-LIBS:texas
-LIBS:intel
-LIBS:audio
-LIBS:interface
-LIBS:digital-audio
-LIBS:philips
-LIBS:display
-LIBS:cypress
-LIBS:siliconi
-LIBS:opto
-LIBS:atmel
-LIBS:contrib
-LIBS:valves
-LIBS:snescart
-LIBS:misc-74
-LIBS:vreg
-LIBS:lpc1754
-LIBS:sd_card
-LIBS:cy62148ev30
-LIBS:mt45w8mw16
-LIBS:cs4344
-LIBS:double_sch_kcom
-LIBS:usb_minib
-LIBS:mic23250
-LIBS:sd2snes-cache
-EELAYER 27 0
+EESchema Schematic File Version 4
+EELAYER 26 0
 EELAYER END
 $Descr A4 11693 8268
@@
 	3500 5150 3500 5300
 Wire Wire Line
-	3500 5300 3300 5300
+	3500 5300 3400 5300
 Connection ~ 3400 5300
 Wire Wire Line
@@
 Connection ~ 4750 4750
 Wire Wire Line
-	4750 4350 4750 5400
+	4750 4350 4750 4650
 Connection ~ 4750 4650
 Wire Wire Line
@@
 	9600 3850 9600 5050
 Wire Wire Line
-	9000 5250 9300 5250
+	9000 5250 9150 5250
 Wire Wire Line
 	9150 5950 9150 6050
@@
 	9150 6050 9600 6050
 Wire Wire Line
-	9600 6350 9600 5450
+	9600 6350 9600 6050
 Connection ~ 9600 6050
 Wire Wire Line
-	7650 2150 7650 1800
-Wire Wire Line
-	9950 2000 7650 2000
-$Comp
-L CY62148EV30-ZSXI U511
+	7650 2150 7650 2000
+Wire Wire Line
+	9950 2000 9600 2000
+$Comp
+L cy62148ev30:CY62148EV30-ZSXI U511
 U 1 1 4D49598F
 P 7650 3450
@@
 Battery power OE switch
 $Comp
-L +3.3V #PWR031
+L power:+3.3V #PWR031
 U 1 1 4BF2FE97
 P 8350 5050
@@
 $EndComp
 $Comp
-L GND #PWR032
+L power:GND #PWR032
 U 1 1 4BF2FE7B
 P 9600 6350
@@
 $EndComp
 $Comp
-L R R511
+L Device:R R511
 U 1 1 4BF2FDAF
 P 9600 3600
@@
 $EndComp
 $Comp
-L R R513
+L Device:R R513
 U 1 1 4BF2FDAC
 P 9150 5700
@@
 $EndComp
 $Comp
-L R R512
+L Device:R R512
 U 1 1 4BF2FDA9
 P 8750 5250
@@
 $EndComp
 $Comp
-L GND #PWR033
+L power:GND #PWR033
 U 1 1 4BF1A006
 P 10500 2000
@@
 $EndComp
 $Comp
-L +BATT #PWR034
+L power:+BATT #PWR034
 U 1 1 4BF19EA4
 P 8400 1400
@@
 $EndComp
 $Comp
-L +3.3V #PWR035
+L power:+3.3V #PWR035
 U 1 1 4BF19E7A
 P 6900 1400
@@
 $EndComp
 $Comp
-L DOUBLE_SCH_KCOM2 D511
+L double_sch_kcom:DOUBLE_SCH_KCOM2 D511
 U 1 1 4BF19DCA
 P 7650 1600
@@
 NoConn ~ 4250 4550
 $Comp
-L GND #PWR036
+L power:GND #PWR036
 U 1 1 4BCA30BF
 P 4750 5400
@@
 ROM_/OE
 $Comp
-L C C502
+L Device:C C502
 U 1 1 4BAD3D55
 P 3550 7000
@@
 $EndComp
 $Comp
-L C C511
+L Device:C C511
 U 1 1 4BAD3D53
 P 10150 2000
@@
 $EndComp
 $Comp
-L C C501
+L Device:C C501
 U 1 1 4BAD3D47
 P 3250 7000
@@
 $EndComp
 $Comp
-L GND #PWR037
+L power:GND #PWR037
 U 1 1 4BAD3D2B
 P 3550 7300
@@
 $EndComp
 $Comp
-L GND #PWR039
+L power:GND #PWR039
 U 1 1 4BAD3D20
 P 3250 7300
@@
 $EndComp
 $Comp
-L +3.3V #PWR040
+L power:+3.3V #PWR040
 U 1 1 4BAD3D0B
 P 3250 6700
@@
 $EndComp
 $Comp
-L GND #PWR041
+L power:GND #PWR041
 U 1 1 4BAD33A7
 P 3400 5400
@@
 $EndComp
 $Comp
-L GND #PWR042
+L power:GND #PWR042
 U 1 1 4BAD339F
 P 7650 5000
@@
 $EndComp
 $Comp
-L +3.3V #PWR044
+L power:+3.3V #PWR044
 U 1 1 4BAD32BE
 P 3500 1550
@@
 128Mbits 70ns PSRAM (ROM area)
 $Comp
-L MT45W8MW16 U501
+L mt45w8mw16:MT45W8MW16 U501
 U 1 1 4B868602
 P 3400 3450
@@
 	1    0    0    -1
 $EndComp
+Wire Wire Line
+	9150 5250 9300 5250
+Wire Wire Line
+	9600 2000 7650 2000
+Wire Wire Line
+	7650 2000 7650 1800
+Wire Wire Line
+	3400 5300 3300 5300
+Wire Wire Line
+	4750 4750 4750 5400
+Wire Wire Line
+	4750 4650 4750 4750
+Wire Wire Line
+	9600 6050 9600 5450
 $EndSCHEMATC
