File: pcb/kicad/RevF/pwr_misc.sch (KiCad schematic (older format))
At the start: 41 parts, among them Q301 IRLML6402PbF, U301 MIC23250-S4YMT, U311 MCP1824-1802E/OT, U321 MCP1824-2502E/OT, U331 PIC12F629-I/P, U341 CS4344

Commit message: S-DD1 + base (trick)
"sd2snes_trick" is the same implementation than "sd2snes_sdd1" but it is
intended to be used as base firmware. It implements S-DD1 core but it is
always disabled. It loads ROMs and runs games perfectly, except for
StarOcean.
"sd2snes_sdd1" corrects BHE and BLE assertion so all accesses from S-DD1
to PSRAM are 16bit wide.
"main.v" simulation is successfull and we get decompressed graphics as
output.
Parts:
- BT351: symbol BATTERY -> Device:Battery
- C301, C302, C303, C304, C311, C312, C321, C322, C331, C332, C333, C341, C342, C343, C344, C345, C346, C347, C348, C349, C391: symbol C -> Device:C
- JP341: symbol JUMPER -> Device:Jumper
- R301, R331, R332, R333, R341, R342, R343, R344: symbol R -> Device:R
- U301: symbol MIC23250_FIXOUT -> mic23250:MIC23250_FIXOUT
- U311, U321: symbol MCP1824-SOT23-Fixed -> vreg:MCP1824-SOT23-Fixed
- U341: symbol CS4344 -> cs4344:CS4344
