File: pcb/kicad/RevF/snesslot.sch (KiCad schematic (older format))
At the start: 42 parts, among them J101 SNESCART_EXT, Q101 2N2222A, U101 74ALVC164245DGG, U102 74ALVC164245DGG, U103 74ALVC164245DGG

Commit message: S-DD1 + base (trick)
"sd2snes_trick" is the same implementation than "sd2snes_sdd1" but it is
intended to be used as base firmware. It implements S-DD1 core but it is
always disabled. It loads ROMs and runs games perfectly, except for
StarOcean.
"sd2snes_sdd1" corrects BHE and BLE assertion so all accesses from S-DD1
to PSRAM are 16bit wide.
"main.v" simulation is successfull and we get decompressed graphics as
output.
Parts:
- C101, C102, C103, C104, C105, C106, C111, C112, C113, C114, C115, C116, C121, C122, C123, C124, C125, C126, C127, C128: symbol C -> Device:C
- J101: symbol SNESCART_EXT -> snescart:SNESCART_EXT
- R101, R102, R103: symbol R -> Device:R
- U101, U102, U103: symbol 74ALVC164245 -> misc-74:74ALVC164245
Connections:
- wire segments 361 -> 425
